Commit message: Reject URDF joints whose axis is missing or of zero length
A movable joint that declares no axis now raises MissingURDFJointAxisError
instead of defaulting to the x-axis, and a zero-length axis raises
ZeroLengthURDFJointAxisError instead of a ValueError. The axes are checked
before the world is built, so the error is raised as itself rather than
wrapped in a BrokenWorldModificationHistoryError.

Co-Authored-By: Claude Opus 5.5 <noreply@anthropic.com>

File: test/semantic_digital_twin_test/test_adapters/dataset/joint_axes.urdf (robot description, URDF)
Before this commit: robot joint_axes, 4 links, 3 joints
Links:
- removed link slider_link
Joints:
- removed joint base_to_slider
